Commit message: added magnetometer and 3D lidar

File: maviss_description/urdf/drone.urdf.xacro (robot description, xacro)
@@ -1,4 +1,4 @@
 <?xml version="1.0"?>
-<robot xmlns:xacro="http://www.ros.org/wiki/xacro" name="maviss_drone">
+<robot xmlns:xacro="http://www.ros.org/wiki/xacro" name="maviss_description">
     <xacro:property name="M_PI" value="3.1415926535897931" />
     <!-- Camera Properties -->
@@ -20,5 +20,5 @@
       <origin rpy="0 0 0" xyz="0   0   0.04"/>
       <geometry>
-        <mesh filename="file://$(find maviss_drone)/meshes/yunque-M.dae"/>
+        <mesh filename="file://$(find maviss_description)/meshes/yunque-M.dae"/>
       </geometry>
     </collision>
@@ -26,5 +26,5 @@
       <origin rpy="0 0 0" xyz="0   0   0.04"/>
       <geometry>
-        <mesh filename="file://$(find maviss_drone)/meshes/yunque-M.dae"/>
+        <mesh filename="file://$(find maviss_description)/meshes/yunque-M.dae"/>
       </geometry>
     </visual>
@@ -105,5 +105,5 @@
       <plugin name='imu' filename='libgazebo_ros_imu_sensor.so'>
         <ros>
-          <namespace>sensor_namespace</namespace>
+          <namespace>imu</namespace>
         </ros>
         <initial_orientation_as_reference>false</initial_orientation_as_reference>
@@ -182,32 +182,39 @@
     </sensor>
   </gazebo>
-  <!--For more details on the structure of gazebo lidar visit https://gazebosim.org/api/sensors/9/classgz_1_1sensors_1_1Lidar.html-->
-  <gazebo reference="lidar_link">
-    <sensor name="lidar" type="ray">
-      <pose>0 0 0 0 0 0</pose>
-      <visualize>true</visualize>
-      <update_rate>20</update_rate>
-      <ray>
-        <scan>
-          <horizontal>
-            <samples>720</samples>
-            <resolution>1</resolution>
-            <min_angle>-1.570796</min_angle>
-            <max_angle>1.570796</max_angle>
-          </horizontal>
-        </scan>
-        <range>
-          <min>0.10</min>
-          <max>30.0</max>
-          <resolution>0.01</resolution>
-        </range>
-      </ray>
-      <plugin name="gazebo_ros_lidar_controller" filename="libgazebo_ros_ray_sensor.so">
-        <ros>
-          <namespace>lidar</namespace>
-          <remapping>~/out:=~/scan</remapping>
-        </ros>
-      </plugin>
-    </sensor>
-  </gazebo>
+ <gazebo reference="lidar_link">
+  <sensor name="lidar" type="ray">
+    <pose>0 0 0 0 0 0</pose>
+    <visualize>false</visualize>
+    <update_rate>20</update_rate>
+    <ray>
+      <scan>
+        <horizontal>
+          <samples>720</samples>
+          <resolution>1</resolution>
+          <min_angle>-3.14159</min_angle>
+          <max_angle>3.14159</max_angle>
+        </horizontal>
+        <vertical>
+          <samples>16</samples>
+          <resolution>1</resolution>
+          <min_angle>-0.2618</min_angle>
+          <max_angle>0.2618</max_angle>
+        </vertical>
+      </scan>
+      <range>
+        <min>0.10</min>
+        <max>30.0</max>
+        <resolution>0.01</resolution>
+      </range>
+    </ray>
+    <plugin name="gazebo_ros_laser_controller" filename="libgazebo_ros_ray_sensor.so">
+      <ros>
+        <namespace>lidar</namespace>
+        <remapping>~/out:=~/points</remapping>
+      </ros>
+      <frame_name>lidar_link</frame_name>
+      <output_type>sensor_msgs/PointCloud2</output_type>
+    </plugin>
+  </sensor>
+ </gazebo>
 </robot>

Commit message: fastlivo added

File: maviss_description/urdf/drone.urdf.xacro (robot description, xacro)
@@ -182,39 +182,8 @@
     </sensor>
   </gazebo>
- <gazebo reference="lidar_link">
-  <sensor name="lidar" type="ray">
-    <pose>0 0 0 0 0 0</pose>
-    <visualize>false</visualize>
-    <update_rate>20</update_rate>
-    <ray>
-      <scan>
-        <horizontal>
-          <samples>720</samples>
-          <resolution>1</resolution>
-          <min_angle>-3.14159</min_angle>
-          <max_angle>3.14159</max_angle>
-        </horizontal>
-        <vertical>
-          <samples>16</samples>
-          <resolution>1</resolution>
-          <min_angle>-0.2618</min_angle>
-          <max_angle>0.2618</max_angle>
-        </vertical>
-      </scan>
-      <range>
-        <min>0.10</min>
-        <max>30.0</max>
-        <resolution>0.01</resolution>
-      </range>
-    </ray>
-    <plugin name="gazebo_ros_laser_controller" filename="libgazebo_ros_ray_sensor.so">
-      <ros>
-        <namespace>lidar</namespace>
-        <remapping>~/out:=~/points</remapping>
-      </ros>
-      <frame_name>lidar_link</frame_name>
-      <output_type>sensor_msgs/PointCloud2</output_type>
-    </plugin>
-  </sensor>
- </gazebo>
+  <!--livox_lidar-->
+  <xacro:include filename="$(find ros2_livox_simulation)/urdf/mid360.xacro" />
+  <xacro:mid360 name="livox" parent="base_link" topic="mid360">
+  <origin xyz="0 0 0.025" rpy="0 0 0"/>
+  </xacro:mid360>
 </robot>

Commit message: gazebo launch file edit

File: maviss_description/urdf/drone.urdf.xacro (robot description, xacro)
@@ -18,5 +18,5 @@
     </inertial>
     <collision name="drone_collision">
-      <origin rpy="0 0 0" xyz="0   0   0.04"/>
+      <origin rpy="0 0 0" xyz="0 0 0"/>
       <geometry>
         <mesh filename="file://$(find maviss_description)/meshes/yunque-M.dae"/>
@@ -24,5 +24,5 @@
     </collision>
     <visual name="drone_visual">
-      <origin rpy="0 0 0" xyz="0   0   0.04"/>
+      <origin rpy="0 0 0" xyz="0 0 0"/>
       <geometry>
         <mesh filename="file://$(find maviss_description)/meshes/yunque-M.dae"/>
@@ -34,10 +34,10 @@
       <origin rpy="0 0 0" xyz="0 0 0"/>
       <geometry>
-        <box size = "0.02 0.02 0.02"/>
+        <box size = "0.0001 0.0001 0.0001"/>
       </geometry>
     </visual>
   </link>
   <joint name="lidar_joint" type="fixed">
-    <origin rpy="0 0 0" xyz="0 0 0"/>
+    <origin rpy="0 0 0" xyz="0.0 0.0 0.3"/>
     <parent link="base_link"/>
     <child link="lidar_link"/>
@@ -94,5 +94,5 @@
           <type>gaussian</type>
           <rate>
-            <mean> 0 </mean>r
+            <mean> 0 </mean>
             <stddev> 0.01 </stddev>
           </rate>
@@ -115,7 +115,7 @@
   <!--Front Camera-->
   <gazebo reference="front_cam">
-    <sensor name="front_camera" type="depth">
+    <sensor name="front_camera" type="camera">
       <always_on>1</always_on>
-      <visualize>1</visualize>
+      <visualize>0</visualize>
       <update_rate>30.0</update_rate>
       <camera>
@@ -145,5 +145,5 @@
     <sensor name="down_camera" type="camera">
       <always_on>1</always_on>
-      <visualize>1</visualize>
+      <visualize>0</visualize>
       <update_rate>30.0</update_rate>
       <camera>
@@ -184,6 +184,6 @@
   <!--livox_lidar-->
   <xacro:include filename="$(find ros2_livox_simulation)/urdf/mid360.xacro" />
-  <xacro:mid360 name="livox" parent="base_link" topic="mid360">
-  <origin xyz="0 0 0.025" rpy="0 0 0"/>
+  <xacro:mid360 name="livox" parent="base_link" topic="livox/lidar">
+  <origin xyz="0 0 0" rpy="0 0 0"/>
   </xacro:mid360>
 </robot>

Commit message: edited livox lidar rotation

File: maviss_description/urdf/drone.urdf.xacro (robot description, xacro)
@@ -30,17 +30,4 @@
     </visual>
   </link>
-  <link name="lidar_link">
-    <visual name="lidar_visual">
-      <origin rpy="0 0 0" xyz="0 0 0"/>
-      <geometry>
-        <box size = "0.0001 0.0001 0.0001"/>
-      </geometry>
-    </visual>
-  </link>
-  <joint name="lidar_joint" type="fixed">
-    <origin rpy="0 0 0" xyz="0.0 0.0 0.3"/>
-    <parent link="base_link"/>
-    <child link="lidar_link"/>
-  </joint>
   <link name="front_cam">
     <visual name="front_cam_visual">
@@ -185,5 +172,5 @@
   <xacro:include filename="$(find ros2_livox_simulation)/urdf/mid360.xacro" />
   <xacro:mid360 name="livox" parent="base_link" topic="livox/lidar">
-  <origin xyz="0 0 0" rpy="0 0 0"/>
+  <origin xyz="0 0 0.3" rpy="${M_PI/2} 0 ${M_PI/2}"/>
   </xacro:mid360>
 </robot>
